Commit message: initial commit for loader gps radar testing

File: ainstein_radar_drivers/urdf/multiple_radars.urdf (robot description, URDF)
Before this commit: robot bobcat, 1 links, 0 joints
Links:
- added link imu_link; visual mesh filename=package://bobcat_o79_testing/meshes/bobcat.stl scale=0.0136 0.0136 0.0136
Joints:
- added joint imu_joint: type fixed, parent base_link, child imu_link, origin xyz=0 0 0 rpy=0 0 0

Commit message: initial commit

File: ainstein_radar_drivers/urdf/multiple_radars.urdf (robot description, URDF)
Before this commit: robot bobcat, 2 links, 1 joints
Links:
- removed link imu_link
- added link lidar_link, mass 1; visual cylinder length=0.1 radius=0.1
Joints:
- removed joint imu_joint
- added joint lidar_joint: type fixed, parent base_link, child lidar_link, origin xyz=0.0 0.0 0.88 rpy=0 0 ${0.0*pi}

Commit message: update for validation test fixture

File: ainstein_radar_drivers/urdf/multiple_radars.urdf (robot description, URDF)
Before this commit: robot bobcat, 2 links, 1 joints
Joints:
- joint lidar_joint: origin xyz=0.0 0.0 0.88 rpy=0 0 ${0.0*pi} -> xyz=0.0 0.0 0.972 rpy=0 0 ${0.0*pi}

Commit message: upadte again for validation fixture

File: ainstein_radar_drivers/urdf/multiple_radars.urdf (robot description, URDF)
Before this commit: robot bobcat, 2 links, 1 joints
Joints:
- joint lidar_joint: origin xyz=0.0 0.0 0.972 rpy=0 0 ${0.0*pi} -> xyz=0.0 0.0 0.968 rpy=0 0 ${0.0*pi}

Commit message: Update CAN node

File: ainstein_radar_drivers/urdf/multiple_radars.urdf (robot description, URDF)
Before this commit: robot bobcat, 2 links, 1 joints
Joints:
- joint lidar_joint: origin xyz=0.0 0.0 0.968 rpy=0 0 ${0.0*pi} -> xyz=0.01 0.0 0.968 rpy=0 0 ${0.0*pi}
